Commit message: feat: update URDF

File: phosphobot/resources/urdf/excavator/simple.urdf (robot description, URDF)
Before this commit: robot excavator, 5 links, 4 joints
Joints:
- joint boom_joint: axis 0 1 0 -> 0 -1 0; limit lower=-1.2 upper=0 effort=1000 velocity=0.5 -> lower=-0.587 upper=0.587 effort=1000 velocity=0.5; origin xyz=0.3 0 0.2 rpy=0 0 0 -> xyz=0.3 0 0.2 rpy=0 -0.46 0
- joint bucket_joint: axis 0 1 0 -> 0 -1 0; limit lower=-1.57 upper=1.57 effort=1000 velocity=0.5 -> lower=0.5 upper=2 effort=1000 velocity=0.5; origin xyz=1.0 0 0 rpy=0 0 0 -> xyz=1.0 0 0 rpy=0 1.916 0
- joint stick_joint: axis 0 1 0 -> 0 -1 0; limit lower=0 upper=1.9 effort=1000 velocity=0.5 -> lower=-1.2 upper=1.5 effort=1000 velocity=0.5; origin xyz=1.5 0 0 rpy=0 0 0 -> xyz=1.5 0 0 rpy=0 1.5 0
