Commit message: Edit urdf limits

File: phosphobot/resources/urdf/piper/urdf/piper.urdf (robot description, URDF)
Before this commit: robot piper, 9 links, 8 joints
Joints:
- joint joint1: limit lower=-2.618 upper=2.618 effort=100 velocity=3 -> lower=-2.6179 upper=2.6179 effort=100 velocity=3
- joint joint3: limit lower=-2.697 upper=0 effort=100 velocity=3 -> lower=-2.967 upper=0 effort=100 velocity=3
- joint joint4: limit lower=-1.832 upper=1.832 effort=100 velocity=3 -> lower=-1.745 upper=1.745 effort=100 velocity=3
- joint joint6: limit lower=-3.14 upper=3.14 effort=100 velocity=3 -> lower=-2.09439 upper=2.09439 effort=100 velocity=3

Commit message: Lower limits

File: phosphobot/resources/urdf/piper/urdf/piper.urdf (robot description, URDF)
Before this commit: robot piper, 9 links, 8 joints
Joints:
- joint joint1: limit lower=-2.6179 upper=2.6179 effort=100 velocity=3 -> lower=-2.6179 upper=2.6179 effort=100 velocity=5
- joint joint2: limit lower=0 upper=3.14 effort=100 velocity=3 -> lower=0 upper=3.14 effort=100 velocity=5
- joint joint4: limit lower=-1.745 upper=1.745 effort=100 velocity=3 -> lower=-1.745 upper=1.745 effort=100 velocity=5
- joint joint5: limit lower=-1.22 upper=1.22 effort=100 velocity=3 -> lower=-1.047 upper=1.047 effort=100 velocity=5
- joint joint7: axis 0 0 -1 -> 0 0 1; limit lower=0 upper=0.04 effort=10 velocity=1 -> lower=0 upper=0.035 effort=10 velocity=1
- joint joint8: axis 0 0 1 -> 0 0 -1; limit lower=-0.04 upper=0 effort=10 velocity=1 -> lower=-0.035 upper=0 effort=10 velocity=1
